File: projects/ANS/cortex-mpu.sch (EAGLE design)
At the start: 7 parts, among them IC1 LM1117MPX-3.3, U1 AT32UC3B164-AUT

Commit message: SPI
Connections:
- net GND: now also U1.GND, U1.GND_2, U1.GND_3
Changed lines of the file:
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@@
 <label x="198.12" y="53.34" size="1.778" layer="95"/>
+</segment>
+<segment>
+<pinref part="U1" gate="A" pin="GND_2"/>
+<wire x1="45.72" y1="91.44" x2="40.64" y2="91.44" width="0.1524" layer="91"/>
+<wire x1="40.64" y1="91.44" x2="40.64" y2="88.9" width="0.1524" layer="91"/>
+<pinref part="U1" gate="A" pin="GND_3"/>
+<wire x1="40.64" y1="88.9" x2="45.72" y2="88.9" width="0.1524" layer="91"/>
+<pinref part="U1" gate="A" pin="GND"/>
+<wire x1="45.72" y1="86.36" x2="40.64" y2="86.36" width="0.1524" layer="91"/>
+<wire x1="40.64" y1="86.36" x2="40.64" y2="88.9" width="0.1524" layer="91"/>
+<junction x="40.64" y="88.9"/>
+<wire x1="40.64" y1="88.9" x2="38.1" y2="88.9" width="0.1524" layer="91"/>
+<label x="33.02" y="88.9" size="1.778" layer="95"/>
 </segment>
 </net>

Commit message: Various Groups
Parts:
- added C3: 100nF, SparkFun-Passives:CAP0603-CAP
- added C4, C5: 22pF, SparkFun-Passives:CAP0603-CAP
- added JP2: (no value), SparkFun-Connectors:M06LOCK_LONGPADS
- added Y1: 7A-16, SparkFun-FreqCtrl:CRYSTALTXC-7A
Connections:
- new net VCC3: C3.2, JP2.1
- net GND: now also C3.1, C4.2, C5.2, JP2.6
- net PA14: now also JP2.4
- net PA15: now also JP2.3
- net PA18: now also C4.1, Y1.1
- net PA19: now also C5.1, Y1.2
- net PA25: now also JP2.5
- net PA9: now also JP2.2
Other:
- note added: "3V3 Regulator"
- note added: "Clock Circuitry"
- note added: "SPI"
- note added: "SPI0_CS2"
- note added: "SPI0_GND"
- note added: "SPI0_MISO"
- note added: "SPI0_MOSI"
- note added: "SPI0_SCK"
- note added: "USB"
- note added: "VCC3"
- moved on the sheet: C1, C2, IC1, JP1, R1, R2, U1

Commit message: Better Grid
Parts:
- added C6, C7: 100nF, SparkFun-Passives:CAP0603-CAP
- added R3, R4: 10k, SparkFun-Passives:RESISTOR0603-RES
- added S1, S2: SWITCH-MOMENTARY-2SMD-4, SparkFun-Electromechanical:SWITCH-MOMENTARY-2SMD-4
Connections:
- new net RESET_N: C6.2, R3.1, S1.1, U1.RESET_N
- net GND: now also C6.1, C7.1, S1.2, S2.2
- net PA13: now also C7.2, R4.1, S2.1
- net VCC3: now also R3.2
Other:
- note added: "JOY Switch"
- note added: "RESET Circuitary"
- moved on the sheet: C1, C4, C5, Y1
