File: projects/ANS/cortex-mpu.sch (EAGLE design)
At the start: 74 parts, among them IC1 LM1117MPX-3.3, U1 AT32UC3B164-AUT, Y1 7A-16

Commit message: Power line
Connections:
- removed net VDDCORE_2: U1.VDDCORE_2
- removed net VDDCORE_3: U1.VDDCORE_3
- net VDDANA: no longer U1.ADVREF, U1.VDDANA
- net VDDCORE: no longer U1.VDDCORE
- net VDDIN: now also U1.ADVREF, U1.VDDANA, U1.VDDIO, U1.VDDIO_2, U1.VDDIO_3
- net VDDIO: no longer U1.VDDIO, U1.VDDIO_2, U1.VDDIO_3
- net VDDOUT: no longer U1.VDDOUT
- net VDDPLL: now also U1.VDDCORE, U1.VDDCORE_2, U1.VDDCORE_3, U1.VDDOUT
Changed lines of the file:
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@@
-</segment>
-</net>
-<net name="VDDCORE_2" class="0">
-<segment>
-<pinref part="U1" gate="A" pin="VDDCORE_2"/>
-<wire x1="20.32" y1="165.1" x2="15.24" y2="165.1" width="0.1524" layer="91"/>
-<label x="5.08" y="165.1" size="1.778" layer="95"/>
-</segment>
-</net>
-<net name="VDDCORE_3" class="0">
-<segment>
-<pinref part="U1" gate="A" pin="VDDCORE_3"/>
-<wire x1="20.32" y1="162.56" x2="15.24" y2="162.56" width="0.1524" layer="91"/>
-<label x="5.08" y="162.56" size="1.778" layer="95"/>
 </segment>
 </net>
 <net name="VDDANA" class="0">
-<segment>
-<pinref part="U1" gate="A" pin="VDDANA"/>
-<wire x1="20.32" y1="167.64" x2="17.78" y2="167.64" width="0.1524" layer="91"/>
-<label x="5.08" y="167.64" size="1.778" layer="95"/>
-<wire x1="17.78" y1="167.64" x2="15.24" y2="167.64" width="0.1524" layer="91"/>
-<wire x1="17.78" y1="167.64" x2="17.78" y2="139.7" width="0.1524" layer="91"/>
-<junction x="17.78" y="167.64"/>
-<pinref part="U1" gate="A" pin="ADVREF"/>
-<wire x1="17.78" y1="139.7" x2="20.32" y2="139.7" width="0.1524" layer="91"/>
-</segment>
 <segment>
 <wire x1="132.08" y1="7.62" x2="132.08" y2="10.16" width="0.1524" layer="91"/>
@@
 </net>
 <net name="VDDCORE" class="0">
-<segment>
-<pinref part="U1" gate="A" pin="VDDCORE"/>
-<wire x1="20.32" y1="160.02" x2="15.24" y2="160.02" width="0.1524" layer="91"/>
-<label x="5.08" y="160.02" size="1.778" layer="95"/>
-</segment>
 <segment>
 <pinref part="C1" gate="G$1" pin="1"/>
@@
 <net name="VDDIN" class="0">
 <segment>
-<pinref part="U1" gate="A" pin="VDDIN"/>
-<wire x1="20.32" y1="157.48" x2="15.24" y2="157.48" width="0.1524" layer="91"/>
-<label x="5.08" y="157.48" size="1.778" layer="95"/>
-</segment>
-<segment>
 <pinref part="C25" gate="G$1" pin="1"/>
 <wire x1="104.14" y1="22.86" x2="104.14" y2="25.4" width="0.1524" layer="91"/>
@@
 <label x="106.68" y="27.94" size="1.778" layer="95"/>
 </segment>
+<segment>
+<pinref part="U1" gate="A" pin="VDDANA"/>
+<wire x1="20.32" y1="167.64" x2="15.24" y2="167.64" width="0.1524" layer="91"/>
+<pinref part="U1" gate="A" pin="VDDIN"/>
+<wire x1="20.32" y1="157.48" x2="15.24" y2="157.48" width="0.1524" layer="91"/>
+<pinref part="U1" gate="A" pin="VDDIO_2"/>
+<wire x1="20.32" y1="154.94" x2="15.24" y2="154.94" width="0.1524" layer="91"/>
+<wire x1="15.24" y1="157.48" x2="15.24" y2="154.94" width="0.1524" layer="91"/>
+<pinref part="U1" gate="A" pin="VDDIO_3"/>
+<wire x1="20.32" y1="152.4" x2="15.24" y2="152.4" width="0.1524" layer="91"/>
+<wire x1="15.24" y1="154.94" x2="15.24" y2="152.4" width="0.1524" layer="91"/>
+<junction x="15.24" y="154.94"/>
+<wire x1="15.24" y1="152.4" x2="15.24" y2="149.86" width="0.1524" layer="91"/>
+<junction x="15.24" y="152.4"/>
+<pinref part="U1" gate="A" pin="VDDIO"/>
+<wire x1="15.24" y1="149.86" x2="20.32" y2="149.86" width="0.1524" layer="91"/>
+<wire x1="15.24" y1="167.64" x2="15.24" y2="157.48" width="0.1524" layer="91"/>
+<junction x="15.24" y="157.48"/>
+<pinref part="U1" gate="A" pin="ADVREF"/>
+<wire x1="20.32" y1="139.7" x2="15.24" y2="139.7" width="0.1524" layer="91"/>
+<wire x1="15.24" y1="139.7" x2="15.24" y2="149.86" width="0.1524" layer="91"/>
+<junction x="15.24" y="149.86"/>
+</segment>
 </net>
 <net name="VDDOUT" class="0">
-<segment>
-<pinref part="U1" gate="A" pin="VDDOUT"/>
-<wire x1="20.32" y1="147.32" x2="15.24" y2="147.32" width="0.1524" layer="91"/>
-<label x="5.08" y="147.32" size="1.778" layer="95"/>
-</segment>
 <segment>
 <pinref part="C22" gate="G$1" pin="1"/>
@@
 <segment>
 <pinref part="U1" gate="A" pin="VDDPLL"/>
-<wire x1="20.32" y1="144.78" x2="15.24" y2="144.78" width="0.1524" layer="91"/>
-<label x="5.08" y="144.78" size="1.778" layer="95"/>
+<wire x1="20.32" y1="144.78" x2="17.78" y2="144.78" width="0.1524" layer="91"/>
+<pinref part="U1" gate="A" pin="VDDOUT"/>
+<wire x1="20.32" y1="147.32" x2="17.78" y2="147.32" width="0.1524" layer="91"/>
+<wire x1="17.78" y1="144.78" x2="17.78" y2="147.32" width="0.1524" layer="91"/>
+<pinref part="U1" gate="A" pin="VDDCORE_2"/>
+<wire x1="20.32" y1="165.1" x2="17.78" y2="165.1" width="0.1524" layer="91"/>
+<pinref part="U1" gate="A" pin="VDDCORE_3"/>
+<wire x1="20.32" y1="162.56" x2="17.78" y2="162.56" width="0.1524" layer="91"/>
+<wire x1="17.78" y1="165.1" x2="17.78" y2="162.56" width="0.1524" layer="91"/>
+<pinref part="U1" gate="A" pin="VDDCORE"/>
+<wire x1="20.32" y1="160.02" x2="17.78" y2="160.02" width="0.1524" layer="91"/>
+<wire x1="17.78" y1="162.56" x2="17.78" y2="160.02" width="0.1524" layer="91"/>
+<junction x="17.78" y="162.56"/>
+<wire x1="17.78" y1="147.32" x2="17.78" y2="160.02" width="0.1524" layer="91"/>
+<junction x="17.78" y="147.32"/>
+<junction x="17.78" y="160.02"/>
 </segment>
 <segment>
@@
 <net name="VDDIO" class="0">
 <segment>
-<pinref part="U1" gate="A" pin="VDDIO_2"/>
-<wire x1="20.32" y1="154.94" x2="15.24" y2="154.94" width="0.1524" layer="91"/>
-<pinref part="U1" gate="A" pin="VDDIO_3"/>
-<wire x1="20.32" y1="152.4" x2="15.24" y2="152.4" width="0.1524" layer="91"/>
-<label x="5.08" y="152.4" size="1.778" layer="95"/>
-<wire x1="15.24" y1="154.94" x2="15.24" y2="152.4" width="0.1524" layer="91"/>
-<pinref part="U1" gate="A" pin="VDDIO"/>
-<wire x1="20.32" y1="149.86" x2="15.24" y2="149.86" width="0.1524" layer="91"/>
-<wire x1="15.24" y1="152.4" x2="15.24" y2="149.86" width="0.1524" layer="91"/>
-<junction x="15.24" y="152.4"/>
-</segment>
-<segment>
 <pinref part="C8" gate="G$1" pin="1"/>

Commit message: Power line
Connections:
- net PA14: now also JP1.5; no longer JP1.4
- net PA16: now also JP1.2
- net PA25: now also JP1.4; no longer JP1.5
- net PA9: no longer JP1.2
- net VCC: now also U1.ADVREF, U1.VDDANA, U1.VDDIN, U1.VDDIO, U1.VDDIO_2, U1.VDDIO_3
- net VDDIN: no longer U1.ADVREF, U1.VDDANA, U1.VDDIN, U1.VDDIO, U1.VDDIO_2, U1.VDDIO_3
Other:
- note added: "SPI0_CS0"
- note removed: "SPI0_CS2"
Changed lines of the file:
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@@
 <part name="SUPPLY5" library="SparkFun-Aesthetics" deviceset="VCC" device=""/>
 <part name="SUPPLY6" library="SparkFun-Aesthetics" deviceset="VCC" device=""/>
+<part name="SUPPLY7" library="SparkFun-Aesthetics" deviceset="VCC" device=""/>
 </parts>
 <sheets>
@@
 <wire x1="264.16" y1="63.5" x2="264.16" y2="96.52" width="0.1524" layer="95"/>
 <wire x1="264.16" y1="96.52" x2="213.36" y2="96.52" width="0.1524" layer="95"/>
-<text x="248.92" y="48.26" size="1.6764" layer="95" align="center-left">SPI0_CS2</text>
+<text x="248.92" y="48.26" size="1.6764" layer="95" align="center-left">SPI0_CS0</text>
 <text x="248.92" y="45.72" size="1.6764" layer="95" align="center-left">SPI0_SCK</text>
 <text x="248.92" y="43.18" size="1.6764" layer="95" align="center-left">SPI0_MISO</text>
@@
 <wire x1="210.82" y1="96.52" x2="210.82" y2="63.5" width="0.1524" layer="95"/>
 <wire x1="210.82" y1="63.5" x2="195.58" y2="63.5" width="0.1524" layer="95"/>
-<wire x1="195.58" y1="63.5" x2="191.24395" y2="59.16395" width="0.1524" layer="95"/>
-<wire x1="191.24395" y1="59.16395" x2="190.5" y2="57.367896875" width="0.1524" layer="95" curve="45.00007"/>
-<wire x1="190.5" y1="57.367896875" x2="190.5" y2="25.4" width="0.1524" layer="95"/>
+<wire x1="195.58" y1="63.5" x2="190.5" y2="58.42" width="0.1524" layer="95"/>
+<wire x1="190.5" y1="58.42" x2="190.5" y2="25.4" width="0.1524" layer="95"/>
 <wire x1="190.5" y1="25.4" x2="152.4" y2="25.4" width="0.1524" layer="95"/>
 <wire x1="152.4" y1="25.4" x2="152.4" y2="96.52" width="0.1524" layer="95"/>
@@
 <instance part="SUPPLY5" gate="G$1" x="200.66" y="78.74"/>
 <instance part="SUPPLY6" gate="G$1" x="236.22" y="35.56" rot="R180"/>
+<instance part="SUPPLY7" gate="G$1" x="10.16" y="162.56"/>
 </instances>
 <busses>
@@
 <wire x1="63.5" y1="134.62" x2="60.96" y2="137.16" width="0.1524" layer="91"/>
 <label x="71.12" y="134.62" size="1.778" layer="95"/>
-</segment>
-<segment>
-<wire x1="213.36" y1="53.34" x2="218.44" y2="53.34" width="0.1524" layer="91"/>
-<wire x1="218.44" y1="53.34" x2="223.52" y2="48.26" width="0.1524" layer="91"/>
-<pinref part="JP1" gate="G$1" pin="2"/>
-<wire x1="223.52" y1="48.26" x2="238.76" y2="48.26" width="0.1524" layer="91"/>
-<label x="213.36" y="53.34" size="1.778" layer="95"/>
 </segment>
 <segment>
@@
 </segment>
 <segment>
-<wire x1="213.36" y1="48.26" x2="218.44" y2="48.26" width="0.1524" layer="91"/>
-<wire x1="218.44" y1="48.26" x2="223.52" y2="43.18" width="0.1524" layer="91"/>
-<pinref part="JP1" gate="G$1" pin="4"/>
-<wire x1="223.52" y1="43.18" x2="238.76" y2="43.18" width="0.1524" layer="91"/>
-<label x="213.36" y="48.26" size="1.778" layer="95"/>
+<wire x1="213.36" y1="45.72" x2="218.44" y2="40.64" width="0.1524" layer="91"/>
+<pinref part="JP1" gate="G$1" pin="5"/>
+<wire x1="218.44" y1="40.64" x2="238.76" y2="40.64" width="0.1524" layer="91"/>
+<label x="218.44" y="40.64" size="1.778" layer="95"/>
 </segment>
 </net>
@@
 </segment>
 <segment>
-<wire x1="213.36" y1="50.8" x2="218.44" y2="50.8" width="0.1524" layer="91"/>
-<wire x1="218.44" y1="50.8" x2="223.52" y2="45.72" width="0.1524" layer="91"/>
+<wire x1="213.36" y1="50.8" x2="218.44" y2="45.72" width="0.1524" layer="91"/>
 <pinref part="JP1" gate="G$1" pin="3"/>
-<wire x1="223.52" y1="45.72" x2="238.76" y2="45.72" width="0.1524" layer="91"/>
-<label x="213.36" y="50.8" size="1.778" layer="95"/>
+<wire x1="218.44" y1="45.72" x2="238.76" y2="45.72" width="0.1524" layer="91"/>
+<label x="218.44" y="45.72" size="1.778" layer="95"/>
 </segment>
 </net>
@@
 <wire x1="63.5" y1="116.84" x2="60.96" y2="119.38" width="0.1524" layer="91"/>
 <label x="71.12" y="116.84" size="1.778" layer="95"/>
+</segment>
+<segment>
+<wire x1="213.36" y1="53.34" x2="218.44" y2="48.26" width="0.1524" layer="91"/>
+<pinref part="JP1" gate="G$1" pin="2"/>
+<wire x1="218.44" y1="48.26" x2="238.76" y2="48.26" width="0.1524" layer="91"/>
+<label x="218.44" y="48.26" size="1.778" layer="95"/>
 </segment>
 </net>
@@
 </segment>
 <segment>
-<wire x1="213.36" y1="45.72" x2="218.44" y2="45.72" width="0.1524" layer="91"/>
-<wire x1="218.44" y1="45.72" x2="223.52" y2="40.64" width="0.1524" layer="91"/>
-<pinref part="JP1" gate="G$1" pin="5"/>
-<wire x1="223.52" y1="40.64" x2="238.76" y2="40.64" width="0.1524" layer="91"/>
-<label x="213.36" y="45.72" size="1.778" layer="95"/>
+<wire x1="213.36" y1="48.26" x2="218.44" y2="43.18" width="0.1524" layer="91"/>
+<pinref part="JP1" gate="G$1" pin="4"/>
+<wire x1="218.44" y1="43.18" x2="238.76" y2="43.18" width="0.1524" layer="91"/>
+<label x="218.44" y="43.18" size="1.778" layer="95"/>
 </segment>
 </net>
@@
 <junction x="236.22" y="50.8"/>
 </segment>
+<segment>
+<pinref part="SUPPLY7" gate="G$1" pin="VCC"/>
+<wire x1="10.16" y1="162.56" x2="10.16" y2="160.02" width="0.1524" layer="91"/>
+<pinref part="U1" gate="A" pin="VDDANA"/>
+<wire x1="20.32" y1="167.64" x2="15.24" y2="167.64" width="0.1524" layer="91"/>
+<pinref part="U1" gate="A" pin="VDDIN"/>
+<wire x1="20.32" y1="157.48" x2="15.24" y2="157.48" width="0.1524" layer="91"/>
+<pinref part="U1" gate="A" pin="VDDIO_2"/>
+<wire x1="20.32" y1="154.94" x2="15.24" y2="154.94" width="0.1524" layer="91"/>
+<wire x1="15.24" y1="157.48" x2="15.24" y2="154.94" width="0.1524" layer="91"/>
+<pinref part="U1" gate="A" pin="VDDIO_3"/>
+<wire x1="20.32" y1="152.4" x2="15.24" y2="152.4" width="0.1524" layer="91"/>
+<wire x1="15.24" y1="154.94" x2="15.24" y2="152.4" width="0.1524" layer="91"/>
+<junction x="15.24" y="154.94"/>
+<wire x1="15.24" y1="152.4" x2="15.24" y2="149.86" width="0.1524" layer="91"/>
+<junction x="15.24" y="152.4"/>
+<pinref part="U1" gate="A" pin="VDDIO"/>
+<wire x1="15.24" y1="149.86" x2="20.32" y2="149.86" width="0.1524" layer="91"/>
+<wire x1="15.24" y1="167.64" x2="15.24" y2="160.02" width="0.1524" layer="91"/>
+<junction x="15.24" y="157.48"/>
+<pinref part="U1" gate="A" pin="ADVREF"/>
+<wire x1="15.24" y1="160.02" x2="15.24" y2="157.48" width="0.1524" layer="91"/>
+<wire x1="20.32" y1="139.7" x2="15.24" y2="139.7" width="0.1524" layer="91"/>
+<wire x1="15.24" y1="139.7" x2="15.24" y2="149.86" width="0.1524" layer="91"/>
+<junction x="15.24" y="149.86"/>
+<wire x1="10.16" y1="160.02" x2="15.24" y2="160.02" width="0.1524" layer="91"/>
+<junction x="15.24" y="160.02"/>
+</segment>
 </net>
 <net name="N$5" class="0">
@@
 <label x="106.68" y="27.94" size="1.778" layer="95"/>
 </segment>
-<segment>
-<pinref part="U1" gate="A" pin="VDDANA"/>
-<wire x1="20.32" y1="167.64" x2="15.24" y2="167.64" width="0.1524" layer="91"/>
-<pinref part="U1" gate="A" pin="VDDIN"/>
-<wire x1="20.32" y1="157.48" x2="15.24" y2="157.48" width="0.1524" layer="91"/>
-<pinref part="U1" gate="A" pin="VDDIO_2"/>
-<wire x1="20.32" y1="154.94" x2="15.24" y2="154.94" width="0.1524" layer="91"/>
-<wire x1="15.24" y1="157.48" x2="15.24" y2="154.94" width="0.1524" layer="91"/>
-<pinref part="U1" gate="A" pin="VDDIO_3"/>
-<wire x1="20.32" y1="152.4" x2="15.24" y2="152.4" width="0.1524" layer="91"/>
-<wire x1="15.24" y1="154.94" x2="15.24" y2="152.4" width="0.1524" layer="91"/>
-<junction x="15.24" y="154.94"/>
-<wire x1="15.24" y1="152.4" x2="15.24" y2="149.86" width="0.1524" layer="91"/>
-<junction x="15.24" y="152.4"/>
-<pinref part="U1" gate="A" pin="VDDIO"/>
-<wire x1="15.24" y1="149.86" x2="20.32" y2="149.86" width="0.1524" layer="91"/>
-<wire x1="15.24" y1="167.64" x2="15.24" y2="157.48" width="0.1524" layer="91"/>
-<junction x="15.24" y="157.48"/>
-<pinref part="U1" gate="A" pin="ADVREF"/>
-<wire x1="20.32" y1="139.7" x2="15.24" y2="139.7" width="0.1524" layer="91"/>
-<wire x1="15.24" y1="139.7" x2="15.24" y2="149.86" width="0.1524" layer="91"/>
-<junction x="15.24" y="149.86"/>
-</segment>
-</net>
+</net>
