File: projects/ANS/cortex-mpu.sch (EAGLE design)
At the start: 71 parts, among them IC1 LM1117MPX-3.3, U1 AT32UC3B164-AUT, Y1 7A-16

Commit message: Fixed consistency
Parts:
- C10: value (none) -> 4.7uF
- C11: value (none) -> 470pF
- C12: value (none) -> 2.2uF
- C13: value (none) -> 1uF
- C14: value (none) -> 10nF
- C8: value (none) -> 100nF
- C9: value (none) -> 1nF
Changed lines of the file:
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@@
 <part name="C6" library="SparkFun-Passives" deviceset="CAP" device="0603-CAP" value="100nF"/>
 <part name="C7" library="SparkFun-Passives" deviceset="CAP" device="0603-CAP" value="100nF"/>
-<part name="C8" library="SparkFun-Passives" deviceset="CAP" device="0603-CAP"/>
-<part name="C9" library="SparkFun-Passives" deviceset="CAP" device="0603-CAP"/>
-<part name="C10" library="SparkFun-Passives" deviceset="CAP" device="0603-CAP"/>
-<part name="C11" library="SparkFun-Passives" deviceset="CAP" device="0603-CAP"/>
-<part name="C12" library="SparkFun-Passives" deviceset="CAP" device="0603-CAP"/>
-<part name="C13" library="SparkFun-Passives" deviceset="CAP" device="0603-CAP"/>
-<part name="C14" library="SparkFun-Passives" deviceset="CAP" device="0603-CAP"/>
+<part name="C8" library="SparkFun-Passives" deviceset="CAP" device="0603-CAP" value="100nF"/>
+<part name="C9" library="SparkFun-Passives" deviceset="CAP" device="0603-CAP" value="1nF"/>
+<part name="C10" library="SparkFun-Passives" deviceset="CAP" device="0603-CAP" value="4.7uF"/>
+<part name="C11" library="SparkFun-Passives" deviceset="CAP" device="0603-CAP" value="470pF"/>
+<part name="C12" library="SparkFun-Passives" deviceset="CAP" device="0603-CAP" value="2.2uF"/>
+<part name="C13" library="SparkFun-Passives" deviceset="CAP" device="0603-CAP" value="1uF"/>
+<part name="C14" library="SparkFun-Passives" deviceset="CAP" device="0603-CAP" value="10nF"/>
 <part name="GND1" library="SparkFun-Aesthetics" deviceset="GND" device=""/>
 <part name="GND2" library="SparkFun-Aesthetics" deviceset="GND" device=""/>
@@
 </sheet>
 </sheets>
+<errors>
+</errors>
 </schematic>
 </drawing>

Commit message: pcb - KINDA
Parts:
- removed PAD1, PAD10, PAD2, PAD3, PAD4, PAD5, PAD6, PAD7, PAD8, PAD9: (no value), wirepad:1,6/0,8
- removed SJ1, SJ2, SJ3, SJ4: JUMPER-PAD-2-NC_BY_TRACE, SparkFun-Passives:JUMPER-PAD-2-NC_BY_TRACE
- removed SJ5: SPK, SparkFun-Passives:JUMPER-PAD-3-2OF3_NC_BY_TRACE_LARGE
- removed SJ6, SJ7: SPK, SparkFun-Passives:JUMPER-PAD-2-NC_BY_TRACE
- added TP1, TP10, TP2, TP3, TP4, TP5, TP6, TP7, TP8, TP9: TEST-POINT2, SparkFun-Passives:TEST-POINT2
- added U$1, U$2, U$3, U$4: JUNCTION, ANS:JUNCTION
- JP2: device SparkFun-Connectors:M06LOCK_LONGPADS -> SparkFun-Connectors:M06LOCK
Connections:
- removed net N$12: SJ5.2, U2.AD0
- removed net N$15: SJ7.2, U2.FSYNC
- removed net N$9: SJ6.2, U2.CLKIN
- net E_SDA: now also TP10.1; no longer PAD10.P
- net GND: now also U2.AD0, U2.CLKIN, U2.FSYNC; no longer SJ5.3, SJ6.1, SJ7.1
- net N$14: now also TP9.1; no longer PAD9.P
- net N$16: now also TP8.1; no longer PAD8.P
- net PA10: now also TP5.1; no longer PAD5.P
- net PA21: now also TP1.1; no longer PAD1.P
- net PA22: now also TP2.1; no longer PAD2.P
- net PA3: now also TP3.1; no longer PAD3.P
- net PA4: now also TP4.1; no longer PAD4.P
- net PA5: now also TP7.1; no longer PAD7.P
- net PA9: now also TP6.1; no longer PAD6.P
- net VCC: no longer SJ5.1
- net VDDCORE0: now also U$1.B; no longer SJ1.1
- net VDDCORE1: now also U$2.B; no longer SJ2.1
- net VDDCORE2: now also U$3.B; no longer SJ3.1
- net VDDOUT: now also U$1.A, U$2.A, U$3.A, U$4.A; no longer SJ1.2, SJ2.2, SJ3.2, SJ4.2
- net VDDPLL: now also U$4.B; no longer SJ4.1
