File: projects/ANS/cortex-mpu-2.brd (EAGLE design)
At the start: 100 x 80 mm, 68 parts, among them IC1 LM1117MPX-3.3, U1 AT32UC3B164-AUT, Y1 7A-16

Commit message: pcb - KINDA
Parts:
- removed SJ1, SJ2, SJ3, SJ4: (no value), SparkFun-Passives:PAD-JUMPER-2-NC_BY_TRACE_YES_SILK
- added U$1, U$2, U$3, U$4: JUNCTION, ANS:JUN-2
- JP2: device SparkFun-Connectors:1X06_LOCK_LONGPADS -> SparkFun-Connectors:1X06_LOCK
- moved D2 14.5 mm to (31.8, 31.8), turned to 270 degrees
- moved TP6 13.5 mm to (31.8, 14.0)
- moved R2 11.7 mm to (38.1, 14.0), turned to 180 degrees
- moved TP5 11.7 mm to (30.5, 14.0)
- moved R1 10.9 mm to (38.1, 11.4), turned to 180 degrees
- moved LOGO1 8.13 mm to (11.4, 36.8)
- moved D5 7.73 mm to (11.4, 25.4)
- moved TP10 7.41 mm to (25.4, 5.08)
- moved TP9 6.35 mm to (27.9, 3.81)
- moved C25 5.68 mm to (35.6, 29.2), turned to 270 degrees
- moved C17 5.68 mm to (31.8, 19.1)
- moved D1 5.24 mm to (11.4, 22.9)
- moved R6 5.24 mm to (21.6, 12.7)
- moved R5 4.02 mm to (6.35, 26.7)
- moved Y1 4.02 mm to (39.4, 26.7)
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Connections:
- net VDDCORE0: now also U$1.B; no longer SJ1.1
- net VDDCORE1: now also U$2.B; no longer SJ2.1
- net VDDCORE2: now also U$3.B; no longer SJ3.1
- net VDDOUT: now also U$1.A, U$2.A, U$3.A, U$4.A; no longer SJ1.2, SJ2.2, SJ3.2, SJ4.2
- net VDDPLL: now also U$4.B; no longer SJ4.1
