File: projects/ANS/cortex-mpu.brd (EAGLE design)
At the start: 100 x 80 mm, 71 parts, among them IC1 LM1117MPX-3.3, U1 AT32UC3B164-AUT, Y1 7A-16

Commit message: brd
Parts:
- moved C22 60.9 mm to (67.3, 68.6), turned to 0 degrees
- moved Y1 56.3 mm to (62.2, 66.0), turned to 90 degrees
- moved C12 56.1 mm to (80.0, 61.0), turned to 180 degrees
- moved PAD8 56.1 mm to (92.7, 31.8), turned to 270 degrees
- moved SJ5 55.1 mm to (74.9, 38.1), turned to 180 degrees
- moved LOGO1 54.4 mm to (62.2, 76.2)
- moved C25 54.3 mm to (67.3, 63.5), turned to 0 degrees
- moved C11 53.4 mm to (80.0, 58.4), turned to 180 degrees
- moved C10 52.8 mm to (76.2, 61.0), turned to 180 degrees
- moved PAD6 51.6 mm to (85.1, 31.8), turned to 270 degrees
- moved PAD7 51.6 mm to (88.9, 31.8), turned to 270 degrees
- moved PAD5 51.6 mm to (81.3, 31.8), turned to 270 degrees
- moved C9 49.9 mm to (76.2, 58.4), turned to 180 degrees
- moved PAD9 49.0 mm to (85.1, 29.2), turned to 90 degrees
- moved C6 47.1 mm to (80.0, 52.1), turned to 270 degrees
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Other:
- board size 100 x 80 mm -> 41.6 x 57.1 mm

Commit message: brd
Parts:
- moved PAD4 28.2 mm to (76.2, 57.1)
- moved PAD3 27.5 mm to (73.7, 57.1)
- moved PAD2 26.8 mm to (71.1, 57.1)
- moved PAD1 26.2 mm to (68.6, 57.1)
- moved PAD8 16.7 mm to (76.2, 34.3), turned to 90 degrees
- moved PAD7 16.3 mm to (76.2, 41.9)
- moved PAD10 12.6 mm to (72.4, 38.1), turned to 0 degrees
- moved PAD9 12.6 mm to (76.2, 38.1), turned to 270 degrees
- moved PAD6 9.67 mm to (76.2, 27.9), turned to 90 degrees
- moved SJ5 8.03 mm to (82.5, 35.6), turned to 90 degrees
- moved C7 7.41 mm to (72.4, 64.8)
- moved C21 6.48 mm to (72.4, 68.6)
- moved C15 5.24 mm to (62.2, 35.6), turned to 180 degrees
- moved C3 5.08 mm to (80.0, 53.3), turned to 180 degrees
- moved C13 5.08 mm to (80.0, 49.5), turned to 180 degrees
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
Commit message: Fixed consistency
Routing:
- net GND: track 0.00 -> 291.1 mm, vias 0 -> 3
- net VCC: track 0.00 -> 140.2 mm, vias 0 -> 4
- net PA14: track 0.00 -> 76.4 mm, vias 0 -> 1
- net PA25: track 0.00 -> 75.4 mm, vias 0 -> 1
- net RESET_N: track 0.00 -> 71.7 mm, vias 0 -> 3
- net PA9: track 0.00 -> 66.8 mm, vias 0 -> 4
- net PA13: track 0.00 -> 64.8 mm, vias 0 -> 2
- net PA26: track 0.00 -> 56.4 mm, vias 0 -> 2
- net DM: track 0.00 -> 44.1 mm, vias 0 -> 4
- net PA16: track 0.00 -> 40.1 mm
- net VBUS: track 0.00 -> 39.3 mm, vias 0 -> 2
- net PA8: track 0.00 -> 38.9 mm, vias 0 -> 2
- net PA18: track 0.00 -> 37.4 mm
- net DP: track 0.00 -> 37.1 mm, vias 0 -> 4
- net PA7: track 0.00 -> 36.5 mm, vias 0 -> 2
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
Commit message: Fixed consistency
Parts:
- turned SJ6 to 90 degrees
Routing:
- net GND: track 291.1 -> 0.00 mm, vias 3 -> 0
- net VCC: track 140.2 -> 0.00 mm, vias 4 -> 0
- net PA14: track 76.4 -> 0.00 mm, vias 1 -> 0
- net PA25: track 75.4 -> 0.00 mm, vias 1 -> 0
- net RESET_N: track 71.7 -> 0.00 mm, vias 3 -> 0
- net PA9: track 66.8 -> 0.00 mm, vias 4 -> 0
- net PA13: track 64.8 -> 0.00 mm, vias 2 -> 0
- net PA26: track 56.4 -> 0.00 mm, vias 2 -> 0
- net DM: track 44.1 -> 0.00 mm, vias 4 -> 0
- net PA16: track 40.1 -> 0.00 mm
- net VBUS: track 39.3 -> 0.00 mm, vias 2 -> 0
- net PA8: track 38.9 -> 0.00 mm, vias 2 -> 0
- net PA18: track 37.4 -> 0.00 mm
- net DP: track 37.1 -> 0.00 mm, vias 4 -> 0
- net PA7: track 36.5 -> 0.00 mm, vias 2 -> 0
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
Commit message: pcb - KINDA
Parts:
- removed PAD1, PAD10, PAD2, PAD3, PAD4, PAD5, PAD6, PAD7, PAD8, PAD9: (no value), wirepad:1,6/0,8
- removed SJ1, SJ2, SJ3, SJ4: (no value), SparkFun-Passives:PAD-JUMPER-2-NC_BY_TRACE_YES_SILK
- removed SJ5: SPK, SparkFun-Passives:PAD-JUMPER-3-2OF3_NC_BY_TRACE_YES_SILK_LARGE
- removed SJ6, SJ7: SPK, SparkFun-Passives:PAD-JUMPER-2-NC_BY_TRACE_YES_SILK
- added TP1, TP10, TP2, TP3, TP4, TP5, TP6, TP7, TP8, TP9: (no value), SparkFun-Passives:PAD.02X.02
- added U$1, U$2, U$3, U$4: JUNCTION, ANS:JUN-2
- JP2: device SparkFun-Connectors:1X06_LOCK_LONGPADS -> SparkFun-Connectors:1X06_LOCK
- moved IC1 148.1 mm to (-48.3, 5.08), turned to 0 degrees
- moved C20 146.4 mm to (-49.5, 45.7)
- moved C19 142.8 mm to (-45.7, 45.7)
- moved S2 139.3 mm to (-44.5, 25.4), turned to 0 degrees
- moved JP1 137.8 mm to (-34.3, 35.6), turned to 0 degrees
- moved C10 135.3 mm to (-57.1, 41.9), turned to 0 degrees
- moved D4 135.0 mm to (-55.9, 35.6), turned to 0 degrees
- moved D3 133.8 mm to (-52.1, 35.6), turned to 0 degrees
- moved R8 133.8 mm to (-57.1, 49.5), turned to 0 degrees
- moved D2 132.6 mm to (-48.3, 35.6), turned to 0 degrees
- moved R7 132.5 mm to (-53.3, 49.5), turned to 0 degrees
- moved D1 131.4 mm to (-44.5, 35.6), turned to 0 degrees
- moved R6 131.3 mm to (-49.5, 49.5), turned to 0 degrees
- moved C9 130.9 mm to (-53.3, 41.9), turned to 0 degrees
- moved S1 130.5 mm to (-34.3, 25.4)
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Connections:
- removed net N$12: SJ5.2, U2.9
- removed net N$15: SJ7.2, U2.11
- removed net N$9: SJ6.2, U2.1
- net E_SDA: now also TP10.P$1; no longer PAD10.1
- net GND: now also U2.1, U2.11, U2.9; no longer SJ5.3, SJ6.1, SJ7.1
- net N$14: now also TP9.P$1; no longer PAD9.1
- net N$16: now also TP8.P$1; no longer PAD8.1
- net PA10: now also TP5.P$1; no longer PAD5.1
- net PA21: now also TP1.P$1; no longer PAD1.1
- net PA22: now also TP2.P$1; no longer PAD2.1
- net PA3: now also TP3.P$1; no longer PAD3.1
- net PA4: now also TP4.P$1; no longer PAD4.1
- net PA5: now also TP7.P$1; no longer PAD7.1
- net PA9: now also TP6.P$1; no longer PAD6.1
- net VCC: no longer SJ5.1
- net VDDCORE0: now also U$1.B; no longer SJ1.1
- net VDDCORE1: now also U$2.B; no longer SJ2.1
- net VDDCORE2: now also U$3.B; no longer SJ3.1
- net VDDOUT: now also U$1.A, U$2.A, U$3.A, U$4.A; no longer SJ1.2, SJ2.2, SJ3.2, SJ4.2
- net VDDPLL: now also U$4.B; no longer SJ4.1
Other:
- board size 41.6 x 57.1 mm -> 100 x 80 mm

Commit message: Schematics - Done
Routing:
- net PA22: track 0.00 -> 3.71 mm
- net PA19: track 0.00 -> 3.61 mm
Changed lines of the file:
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@@
 <contactref element="C25" pad="1"/>
 <wire x1="-41.22" y1="35.56" x2="-23.71" y2="49.53" width="0" layer="19" extent="1-1"/>
-<wire x1="34.5948" y1="29.464" x2="-41.22" y2="35.56" width="0" layer="19" extent="1-1"/>
+<wire x1="34.5948" y1="29.464" x2="37.846" y2="29.464" width="0.3048" layer="1"/>
+<wire x1="37.846" y1="29.464" x2="38.1" y2="29.21" width="0.3048" layer="1"/>
+<wire x1="38.1" y1="29.21" x2="-23.71" y2="49.53" width="0" layer="19" extent="1-16"/>
 </signal>
 <signal name="PA20">
@@
 <contactref element="D4" pad="C"/>
 <contactref element="TP2" pad="P$1"/>
-<wire x1="-55.88" y1="36.437" x2="34.5948" y2="30.9626" width="0" layer="19" extent="1-1"/>
 <wire x1="-46.99" y1="52.07" x2="-55.88" y2="36.437" width="0" layer="19" extent="1-1"/>
+<wire x1="34.5948" y1="30.9626" x2="37.6174" y2="30.9626" width="0.3048" layer="1"/>
+<wire x1="37.6174" y1="30.9626" x2="38.1" y2="30.48" width="0.4064" layer="1"/>
+<wire x1="38.1" y1="30.48" x2="-46.99" y2="52.07" width="0" layer="19" extent="1-16"/>
 </signal>
 <signal name="PA23">
@@
 <wire x1="-23.71" y1="45.72" x2="-27.52" y2="45.72" width="0" layer="19" extent="1-1"/>
 </signal>
+<signal name="N$9">
+<via x="38.1" y="30.48" extent="1-16" drill="0.5" diameter="0.254" shape="octagon"/>
+</signal>
+<signal name="N$12">
+<via x="38.1" y="29.21" extent="1-16" drill="0.5" diameter="0.254" shape="octagon"/>
+</signal>
+<signal name="N$13">
+<via x="38.1" y="27.94" extent="1-16" drill="0.5" diameter="0.254" shape="octagon"/>
+</signal>
 </signals>

Commit message: Fixed consistency
Parts:
- added C26, C27, C28: (no value), SparkFun-Passives:0603-CAP
- added R13, R14: 10kR, SparkFun-Passives:0603-RES
- added U$5: MPU-9250, SparkFun-Sensors:QFN-24-NP
- moved TP4 113.6 mm to (50.8, 3.81)
- moved TP3 110.6 mm to (53.3, 11.4)
- moved TP2 102.4 mm to (50.8, 21.6)
- moved TP1 91.5 mm to (44.5, 30.5)
- moved TP6 90.3 mm to (24.1, 12.7)
- moved TP5 84.6 mm to (21.6, 15.2)
- moved C10 82.4 mm to (21.6, 17.8), flipped to the bottom, turned to 90 degrees
- moved C18 79.1 mm to (26.7, 6.35), turned to 90 degrees
- moved C9 77.5 mm to (20.3, 17.8), flipped to the bottom, turned to 90 degrees
- moved C17 73.4 mm to (25.4, 8.89), turned to 270 degrees
- moved C7 71.8 mm to (24.1, 25.4), flipped to the bottom
- moved R2 71.2 mm to (26.7, 12.7), turned to 270 degrees
- moved C8 70.3 mm to (16.5, 17.8), flipped to the bottom, turned to 90 degrees
- moved C6 70.3 mm to (24.1, 17.8), flipped to the bottom, turned to 90 degrees
- moved U$4 68.2 mm to (20.3, 24.1), turned to 180 degrees
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Connections:
- new net N$15: R13.2, R14.2
- new net N$17: C28.1, U$5.10
- new net N$18: C27.1, U$5.13
- new net N$19: C26.1, U$5.8
- net PA10: now also R14.1, U$5.24
- net PA5: now also U$5.12
- net PA9: now also R13.1, U$5.23
Routing:
- net GND: track 0.00 -> 64.9 mm, vias 0 -> 4
- net VDDOUT: track 0.00 -> 22.9 mm, vias 0 -> 1
- net PA9: track 0.00 -> 16.5 mm
- net PA10: track 0.00 -> 15.6 mm, vias 0 -> 2
- net VDDCORE2: track 0.00 -> 12.9 mm, vias 0 -> 1
- net VDDCORE0: track 0.00 -> 11.2 mm, vias 0 -> 1
- net VCC: track 0.00 -> 10.8 mm
- net VDDIN: track 0.00 -> 9.85 mm, vias 0 -> 1
- net VDDCORE1: track 0.00 -> 9.42 mm, vias 0 -> 1
- net VDDPLL: track 0.00 -> 8.51 mm, vias 0 -> 1
- net ADVREF: track 0.00 -> 7.11 mm, vias 0 -> 1
- net VDDIO0: track 0.00 -> 6.55 mm, vias 0 -> 1
- net VDDIO1: track 0.00 -> 6.16 mm, vias 0 -> 1
- net VDDANA: track 0.00 -> 5.52 mm, vias 0 -> 1
- net VDDIO2: track 0.00 -> 5.28 mm, vias 0 -> 1
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
Commit message: Fixed consistency
Parts:
- removed C15: 10nF, SparkFun-Passives:0603-CAP
- removed C16, C18: 0.1uF, SparkFun-Passives:0603-CAP
- removed C17: 2.2nF, SparkFun-Passives:0603-CAP
- removed R1, R2: 10kR, SparkFun-Passives:0603-RES
- removed TP10, TP8, TP9: (no value), SparkFun-Passives:PAD.02X.02
- removed U2: (no value), SparkFun-Sensors:QFN-24-NP
- C26: value (none) -> 10nF
- C27, C28: value (none) -> 0.1uF
- moved R14 98.0 mm to (29.2, 8.89)
- moved R13 97.7 mm to (29.2, 11.4)
- moved U$5 86.4 mm to (21.6, 6.35)
- moved C28 78.0 mm to (10.2, 8.89)
- moved C26 77.6 mm to (11.4, 1.27)
- moved C27 76.9 mm to (10.2, 5.08)
- moved TP6 5.24 mm to (29.2, 14.0)
- moved TP5 2.54 mm to (21.6, 12.7)
Connections:
- removed net E_SDA: TP10.P$1, U2.6
- removed net N$10: C18.1, U2.10
- removed net N$11: C17.1, U2.20
- removed net N$14: TP9.P$1, U2.7
- removed net N$15: R13.2, R14.2
- removed net N$16: TP8.P$1, U2.22
- removed net N$18: C27.1, U$5.13
- removed net N$19: C26.1, U$5.8
- net GND: now also C26.2, C27.2, C28.2, U$5.11, U$5.18, U$5.20, U$5.9; no longer C15.2, C16.2, C17.2, C18.2, U2.1, U2.11, U2.15, U2.17, U2.18, U2.9
- net PA10: now also TP6.P$1; no longer R1.1, TP5.P$1, U2.24
- net PA5: no longer U2.12
- net PA9: now also TP5.P$1; no longer R2.1, TP6.P$1, U2.23
- net VCC: now also C26.1, C27.1, R13.2, R14.2, U$5.1, U$5.13, U$5.22, U$5.8; no longer C15.1, C16.1, R1.2, R2.2, U2.13, U2.3, U2.8
Routing:
- net GND: track 64.9 -> 44.7 mm
- net PA9: track 16.5 -> 0.00 mm
- net PA10: track 15.6 -> 0.00 mm, vias 2 -> 0
- net VCC: track 10.8 -> 0.00 mm
- net N$14: track 2.78 -> 0.00 mm
- net N$16: track 1.91 -> 0.00 mm
- net E_SDA: track 1.82 -> 0.00 mm
