File: projects/ANS/cortex-mpu.brd (EAGLE design)
At the start: 100 x 80 mm, 64 parts, among them IC1 LM1117MPX-3.3, U1 AT32UC3B164-AUT, Y1 7A-16

Commit message: bOARD
Parts:
- moved C28 14.2 mm to (22.9, 2.54), turned to 180 degrees
- moved R13 10.5 mm to (26.7, 1.27), turned to 180 degrees
- moved C27 9.25 mm to (19.1, 2.54)
- moved TP4 8.13 mm to (45.7, 10.2)
- moved C26 7.62 mm to (19.1, 1.27)
- moved R14 6.84 mm to (26.7, 2.54), turned to 180 degrees
- moved TP6 5.08 mm to (24.1, 14.0)
- moved U$5 1.27 mm to (21.6, 7.62)
- moved TP5 1.27 mm to (22.9, 12.7)
Routing:
- net VCC: track 0.00 -> 29.3 mm
- net GND: track 44.7 -> 61.5 mm
- net PA10: track 0.00 -> 5.84 mm
- net PA9: track 0.00 -> 5.51 mm
- net N$17: track 0.00 -> 3.85 mm
Other:
- board size 100 x 80 mm -> 100 x 82.5 mm

Commit message: Board
Parts:
- JP2: value (none) -> FEMALE 2x3; device SparkFun-Connectors:1X06_LOCK -> SparkFun-Connectors:2X3
- moved C22 97.6 mm to (35.6, 15.2)
- moved R8 95.2 mm to (34.3, 22.9)
- moved R7 92.0 mm to (34.3, 21.6)
- moved D4 87.3 mm to (30.5, 22.9), turned to 90 degrees
- moved C19 84.1 mm to (29.7, 8.44), flipped to the bottom, turned to 45 degrees
- moved D3 83.7 mm to (30.5, 21.6), turned to 90 degrees
- moved R4 83.0 mm to (31.1, 10.2), flipped to the bottom, turned to 225 degrees
- moved C20 81.8 mm to (27.3, 17.8), flipped to the bottom, turned to 90 degrees
- moved S2 80.7 mm to (36.2, 22.9), flipped to the bottom
- moved R6 78.2 mm to (16.5, 7.62), turned to 270 degrees
- moved R3 74.4 mm to (29.2, 17.8), flipped to the bottom, turned to 270 degrees
- moved Y1 73.6 mm to (31.8, 16.5), turned to 270 degrees
- moved S1 71.1 mm to (36.2, 15.9), flipped to the bottom
- moved C23 70.3 mm to (38.7, 4.45), flipped to the bottom, turned to 270 degrees
- moved D2 70.3 mm to (17.8, 11.4), turned to 315 degrees
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Routing:
- net GND: track 61.5 -> 172.2 mm, vias 4 -> 5
- net VCC: track 29.3 -> 110.4 mm, vias 0 -> 1
- net PA25: track 0.00 -> 49.9 mm
- net RESET_N: track 0.00 -> 33.8 mm, vias 0 -> 1
- net PA5: track 0.00 -> 32.9 mm, vias 0 -> 2
- net PA26: track 0.00 -> 25.4 mm, vias 0 -> 1
- net PA14: track 0.00 -> 24.1 mm
- net PA16: track 0.00 -> 23.3 mm
- net PA10: track 5.84 -> 29.0 mm, vias 0 -> 2
- net PA9: track 5.51 -> 28.5 mm
- net PA15: track 0.00 -> 22.3 mm
- net PA13: track 0.00 -> 19.9 mm, vias 0 -> 1
- net PA18: track 0.00 -> 17.7 mm
- net PA19: track 0.00 -> 14.5 mm
- net DM: track 0.00 -> 9.59 mm
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
Commit message: Board layout
Parts:
- moved R10 28.4 mm to (27.9, 28.6)
- moved D6 24.5 mm to (24.8, 28.6), turned to 90 degrees
- moved C21 9.09 mm to (14.0, 10.8), flipped to the bottom
- moved R5 4.58 mm to (11.4, 16.5), turned to 270 degrees
- moved C24 4.26 mm to (10.2, 10.8), flipped to the bottom, turned to 270 degrees
- moved R9 4.02 mm to (8.89, 16.5), turned to 270 degrees
- moved IC1 3.24 mm to (12.1, 4.45), flipped to the bottom, turned to 180 degrees
Routing:
- net VBUS: track 6.52 -> 83.6 mm, vias 1 -> 2
- net VCC: track 110.4 -> 157.6 mm, vias 1 -> 3
- net GND: track 172.2 -> 205.9 mm
- net N$8: track 2.08 -> 3.88 mm
- net N$5: track 0.00 -> 1.45 mm

Commit message: Board layout
Parts:
- moved LOGO1 31.0 mm to (36.5, 31.8)
Other:
- board size 100 x 82.5 mm -> 34.3 x 40 mm
- board text added: "WARNING This part of the board may get very hot."
Changed lines of the file:
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@@
 <layer number="110" name="fp0" color="7" fill="1" visible="no" active="yes"/>
 <layer number="111" name="LPC17xx" color="7" fill="1" visible="no" active="yes"/>
-<layer number="112" name="tSilk" color="7" fill="1" visible="no" active="yes"/>
+<layer number="112" name="tSilk" color="7" fill="1" visible="yes" active="yes"/>
 <layer number="113" name="IDFDebug" color="4" fill="1" visible="no" active="yes"/>
 <layer number="116" name="Patch_BOT" color="9" fill="4" visible="no" active="yes"/>
@@
 <board>
 <plain>
-<wire x1="0" y1="-2.54" x2="100" y2="-2.54" width="0" layer="20"/>
-<wire x1="100" y1="-2.54" x2="100" y2="80" width="0" layer="20"/>
-<wire x1="100" y1="80" x2="0" y2="80" width="0" layer="20"/>
-<wire x1="0" y1="80" x2="0" y2="-2.54" width="0" layer="20"/>
+<wire x1="38.985475" y1="37.465" x2="26.933025" y2="37.465" width="0" layer="20"/>
+<wire x1="26.933025" y1="37.465" x2="26.035" y2="36.566975" width="0" layer="20"/>
+<wire x1="26.035" y1="36.566975" x2="26.035" y2="35.823025" width="0" layer="20"/>
+<wire x1="26.035" y1="35.823025" x2="25.136975" y2="34.925" width="0" layer="20"/>
+<wire x1="25.136975" y1="34.925" x2="9.274525" y2="34.925" width="0" layer="20"/>
+<wire x1="9.274525" y1="34.925" x2="6.985" y2="32.635475" width="0" layer="20"/>
+<wire x1="6.985" y1="32.635475" x2="6.985" y2="0.078171875" width="0" layer="20"/>
+<wire x1="6.985" y1="0.078171875" x2="9.603171875" y2="-2.54" width="0" layer="20"/>
+<wire x1="9.603171875" y1="-2.54" x2="38.580925" y2="-2.54" width="0" layer="20"/>
+<wire x1="38.580925" y1="-2.54" x2="41.275" y2="0.154075" width="0" layer="20"/>
+<wire x1="41.275" y1="0.154075" x2="41.275" y2="35.175475" width="0" layer="20"/>
+<wire x1="41.275" y1="35.175475" x2="38.985475" y2="37.465" width="0" layer="20"/>
+<text x="10.16" y="5.08" size="0.6096" layer="112" font="vector" ratio="15" rot="R90" align="center">WARNING
+This part of the board
+may get very hot.</text>
+<hole x="10.16" y="33.02" drill="0.508"/>
+<hole x="8.89" y="31.75" drill="0.508"/>
+<hole x="9.525" y="0" drill="0.508"/>
 </plain>
 <attributes>
@@
 </element>
 <element name="L1" library="SparkFun-Passives" package="0603" value="3.3uH" x="13.97" y="12.7" rot="R45"/>
-<element name="LOGO1" library="SparkFun-Aesthetics" package="OSHW-LOGO-S_COPPER" value="OSHW-LOGOS-COPPER" x="7.925" y="43.84"/>
+<element name="LOGO1" library="SparkFun-Aesthetics" package="OSHW-LOGO-S_COPPER" value="OSHW-LOGOS-COPPER" x="36.5" y="31.775"/>
 <element name="R10" library="SparkFun-Passives" package="0603-RES" value="1kR" x="27.94" y="28.575"/>
 <element name="R11" library="SparkFun-Passives" package="0603-RES" value="39R" x="27.94" y="29.845" rot="R180"/>
@@
 </board>
 </drawing>
+<compatibility>
+<note version="6.3" minversion="6.2.2" severity="warning">
+Since Version 6.2.2 text objects can contain more than one line,
+which will not be processed correctly with this version.
+</note>
+</compatibility>
 </eagle>

Commit message: DONE
Routing:
- added copper zone on layer 1, net GND
- added copper zone on layer 16, net GND
- added copper zone on layer 1, net VCC
- added copper zone on layer 16, net VCC
Other:
- outline, holes or cut-outs redrawn
- board text added: "5v"
- board text added: "GND"

Commit message: DONE
Other:
- board text added: "AT32UC3B"
- board text added: "MPU-9250"
- board text added: "SPIO"
- board text added: "This part of the board may get very hot."
- board text removed: "WARNING This part of the board may get very hot."
Changed lines of the file:
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@@
 <wire x1="41.275" y1="0.154075" x2="41.275" y2="35.175475" width="0" layer="20"/>
 <wire x1="41.275" y1="35.175475" x2="38.985475" y2="37.465" width="0" layer="20"/>
-<text x="12.065" y="3.81" size="0.6096" layer="104" font="vector" ratio="15" rot="R90" align="center">WARNING
-This part of the board
+<text x="12.065" y="3.81" size="0.6096" layer="21" font="vector" ratio="15" rot="R90" align="center">This part of the board
 may get very hot.</text>
 <hole x="10.16" y="33.02" drill="0.508"/>
@@
 <text x="33.655" y="34.925" size="1.016" layer="104" font="vector" ratio="15" align="center">5v</text>
 <text x="26.035" y="34.925" size="1.016" layer="104" font="vector" ratio="15" align="center">GND</text>
+<wire x1="4.445" y1="3.81" x2="2.54" y2="0.635" width="0.4064" layer="21"/>
+<wire x1="2.54" y1="0.635" x2="6.35" y2="0.635" width="0.4064" layer="21"/>
+<wire x1="6.35" y1="0.635" x2="4.445" y2="3.81" width="0.4064" layer="21"/>
+<text x="15.24" y="28.575" size="1.016" layer="21">AT32UC3B</text>
+<text x="17.78" y="3.81" size="1.016" layer="21">MPU-9250</text>
+<text x="34.925" y="10.16" size="1.27" layer="21" align="center">SPIO</text>
 </plain>
 <attributes>
@@
 <vertex x="24.13" y="34.29"/>
 </polygon>
+<wire x1="20.32" y1="2.54" x2="19.9" y2="2.54" width="0" layer="19" extent="1-1"/>
+<wire x1="36.41" y1="17.78" x2="35.27" y2="18.125" width="0" layer="19" extent="1-16"/>
 </signal>
 <signal name="VBUS">

Commit message: Fix
Parts:
- added U$6: (no value), SparkFun-Aesthetics:OSHW-LOGO-L
- added U$7: (no value), SparkFun-Aesthetics:OSHW-LOGO-S
- moved LOGO1 0.97 mm to (37.5, 31.8)
Other:
- board text added: "OpenSourceHardware github.com/prashnts"
- board text added: "This part may get very hot"
- board text added: "USB"
- board text added: "WGB v0.1"
- board text removed: "This part of the board may get very hot."
Changed lines of the file:
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@@
 <wire x1="41.275" y1="0.154075" x2="41.275" y2="35.175475" width="0" layer="20"/>
 <wire x1="41.275" y1="35.175475" x2="38.985475" y2="37.465" width="0" layer="20"/>
-<text x="12.065" y="3.81" size="0.6096" layer="21" font="vector" ratio="15" rot="R90" align="center">This part of the board
-may get very hot.</text>
 <hole x="10.16" y="33.02" drill="0.508"/>
 <hole x="8.89" y="31.75" drill="0.508"/>
@@
 <text x="33.655" y="34.925" size="1.016" layer="104" font="vector" ratio="15" align="center">5v</text>
 <text x="26.035" y="34.925" size="1.016" layer="104" font="vector" ratio="15" align="center">GND</text>
-<wire x1="4.445" y1="3.81" x2="2.54" y2="0.635" width="0.4064" layer="21"/>
-<wire x1="2.54" y1="0.635" x2="6.35" y2="0.635" width="0.4064" layer="21"/>
-<wire x1="6.35" y1="0.635" x2="4.445" y2="3.81" width="0.4064" layer="21"/>
 <text x="15.24" y="28.575" size="1.016" layer="21">AT32UC3B</text>
 <text x="17.78" y="3.81" size="1.016" layer="21">MPU-9250</text>
 <text x="34.925" y="10.16" size="1.27" layer="21" align="center">SPIO</text>
+<text x="8.255" y="26.035" size="1.27" layer="21" rot="R90" align="center">WGB v0.1</text>
+<text x="24.765" y="-0.635" size="0.6096" layer="21" rot="R180" align="center">OpenSourceHardware
+github.com/prashnts</text>
+<text x="34.925" y="31.75" size="0.8128" layer="21" rot="R90" align="center">USB</text>
+<text x="12.065" y="4.445" size="0.6096" layer="21" rot="R270" align="center">This part
+may get
+very hot</text>
 </plain>
 <attributes>
@@
 </element>
 <element name="L1" library="SparkFun-Passives" package="0603" value="3.3uH" x="13.97" y="12.7" rot="R45"/>
-<element name="LOGO1" library="SparkFun-Aesthetics" package="OSHW-LOGO-S_COPPER" value="OSHW-LOGOS-COPPER" x="36.5" y="31.775"/>
+<element name="LOGO1" library="SparkFun-Aesthetics" package="OSHW-LOGO-S_COPPER" value="OSHW-LOGOS-COPPER" x="37.465" y="31.75"/>
 <element name="R10" library="SparkFun-Passives" package="0603-RES" value="1kR" x="27.94" y="28.575"/>
 <element name="R11" library="SparkFun-Passives" package="0603-RES" value="39R" x="27.94" y="29.845" rot="R180"/>
@@
 <element name="R13" library="SparkFun-Passives" package="0603-RES" value="10kR" x="26.67" y="2.54" rot="R180"/>
 <element name="R14" library="SparkFun-Passives" package="0603-RES" value="10kR" x="26.67" y="1.27" rot="R180"/>
+<element name="U$6" library="SparkFun-Aesthetics" package="OSHW-LOGO-L" value="" x="12.7" y="29.21" rot="MR0"/>
+<element name="U$7" library="SparkFun-Aesthetics" package="OSHW-LOGO-S" value="" x="37.465" y="31.75"/>
 </elements>
 <signals>

Commit message: Fixed OSH logo
Parts:
- moved U$6 24.8 mm to (12.7, 4.45)
Changed lines of the file:
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@@
 <element name="R13" library="SparkFun-Passives" package="0603-RES" value="10kR" x="26.67" y="2.54" rot="R180"/>
 <element name="R14" library="SparkFun-Passives" package="0603-RES" value="10kR" x="26.67" y="1.27" rot="R180"/>
-<element name="U$6" library="SparkFun-Aesthetics" package="OSHW-LOGO-L" value="" x="12.7" y="29.21" rot="MR0"/>
+<element name="U$6" library="SparkFun-Aesthetics" package="OSHW-LOGO-L" value="" x="12.7" y="4.445" rot="MR0"/>
 <element name="U$7" library="SparkFun-Aesthetics" package="OSHW-LOGO-S" value="" x="37.465" y="31.75"/>
 </elements>
